File: BUCK_MC34063_STEP_DOWN_3.3_v1_1.kicad_sch (KiCad schematic)
At the start: 9 parts, among them U5 MC34063AD_copy

Commit message: added footprints
Parts:
- R32: footprint Resistor_SMD:R_0805_2012Metric_Pad1.15x1.40mm_HandSolder -> (none)
Changed lines of the file:
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@@
     (property "Reference" "R32" (id 0) (at 169.0878 82.55 90))
     (property "Value" "0R18" (id 1) (at 166.7764 82.55 90))
-    (property "Footprint" "Resistor_SMD:R_0805_2012Metric_Pad1.15x1.40mm_HandSolder" (id 2) (at 162.052 82.55 90)
+    (property "Footprint" "" (id 2) (at 162.052 82.55 90)
       (effects (font (size 1.27 1.27)) hide)
     )
