File: NMOS_DRIVER.kicad_sch (KiCad schematic)
At the start: 6 parts, among them Q2 Q_NPN_BEC, Q3 Q_NMOS_GDS

Commit message: added footprints
Parts:
- R26, R27, R_D1, R_P1: footprint Resistor_SMD:R_0805_2012Metric_Pad1.15x1.40mm_HandSolder -> (none)
Changed lines of the file:
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@@
     (property "Reference" "R_P1" (id 0) (at 86.36 86.36 90))
     (property "Value" "R" (id 1) (at 86.36 83.4136 90))
-    (property "Footprint" "Resistor_SMD:R_0805_2012Metric_Pad1.15x1.40mm_HandSolder" (id 2) (at 86.36 84.582 90)
+    (property "Footprint" "" (id 2) (at 86.36 84.582 90)
       (effects (font (size 1.27 1.27)) hide)
     )
@@
       (effects (font (size 1.27 1.27)) (justify left))
     )
-    (property "Footprint" "Resistor_SMD:R_0805_2012Metric_Pad1.15x1.40mm_HandSolder" (id 2) (at 99.822 68.58 90)
+    (property "Footprint" "" (id 2) (at 99.822 68.58 90)
       (effects (font (size 1.27 1.27)) hide)
     )
@@
       (effects (font (size 1.27 1.27)) (justify left))
     )
-    (property "Footprint" "Resistor_SMD:R_0805_2012Metric_Pad1.15x1.40mm_HandSolder" (id 2) (at 118.872 68.58 90)
+    (property "Footprint" "" (id 2) (at 118.872 68.58 90)
       (effects (font (size 1.27 1.27)) hide)
     )
@@
     (property "Reference" "R_D1" (id 0) (at 86.36 80.01 90))
     (property "Value" "R" (id 1) (at 86.36 77.0636 90))
-    (property "Footprint" "Resistor_SMD:R_0805_2012Metric_Pad1.15x1.40mm_HandSolder" (id 2) (at 86.36 78.232 90)
+    (property "Footprint" "" (id 2) (at 86.36 78.232 90)
       (effects (font (size 1.27 1.27)) hide)
     )
